File: FRDMK64F_Shield/FRDMK64F_Shield.kicad_pcb (KiCad board)
At the start: 2 copper layers, 18 parts, among them J1 CONN_02X08, J2 CONN_02X10, J3 CONN_02X08, J4 CONN_02X06

Commit message: Avances en el pcb
Parts:
- moved CINTA1 90.2 mm to (148.6, 40.6), turned to 180 degrees
- moved ULTRASONIC_1 65.2 mm to (114.3, 49.5)
- moved ENABLED1 62.6 mm to (128.3, 45.7)
- moved HORN1 59.4 mm to (152.4, 45.7)
- moved HALL_5 55.8 mm to (114.3, 61.0), turned to 90 degrees
- moved BATTERY1 55.3 mm to (174.0, 55.9)
- moved HALL_4 52.8 mm to (114.3, 64.8), turned to 90 degrees
- moved POWER1 49.8 mm to (174.0, 62.2)
- moved HALL_3 44.7 mm to (114.3, 76.2), turned to 90 degrees
- moved HALL_2 42.4 mm to (114.3, 80.0), turned to 90 degrees
- moved HALL_1 39.6 mm to (114.3, 85.1), turned to 90 degrees
- moved HALL_0 37.8 mm to (114.3, 88.9), turned to 90 degrees
- moved BREAK1 35.7 mm to (125.7, 77.5)
- moved ULTRASONIC_2 31.6 mm to (118.1, 96.5), turned to 180 degrees
- moved J1 30.6 mm to (138.4, 50.8)
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Routing:
- net /HALL0_INT: track 0.00 -> 21.3 mm
- net /ULTRA2_ECHO: track 0.00 -> 21.0 mm
- net /ULTRA2_TRIG: track 0.00 -> 20.6 mm
- net /HALL1_INT: track 0.00 -> 20.6 mm
- net /HALL2_INT: track 0.00 -> 20.4 mm
- net /BATTERY: track 0.00 -> 17.3 mm
- net /POWER: track 0.00 -> 15.9 mm
- net /HORN: track 0.00 -> 13.9 mm
